File: Precharge_Nauka.kicad_sch (KiCad schematic)
At the start: 244 parts, among them J1 Conn_02x03_Top_Bottom, J2 Conn_01x01, J3 Conn_01x01, J4 Conn_01x01, Q1 2N7002, Q2 C2M0280120D, Q3 C2M0280120D, Q4 C2M0280120D, Q5 C2M0280120D, Q6 2N7002, U1 TS3702IDT, U2 LMV321IDBVR, U3 74LVC1G08, U4 LMV321IDBVR, U5 PC817

Commit message: VER1.0: уместил в прямоугольник все, заменил операционники измерительные
Parts:
- removed U2, U4: LMV321IDBVR, Package_TO_SOT_SMD:SOT-23-5, symbol Amplifier_Operational:LMV321
- added U6, U7: OPA333xxDBV, Package_TO_SOT_SMD:SOT-23-5, symbol Amplifier_Operational:OPA333xxDBV
Connections:
- net +5V: now also U6.5 (V+), U7.5 (V+)
- net GND1: now also U6.2 (V-), U7.2 (V-)
- net at C21.2, R21.1, R26.2: now also U7.1
- net at C3.2, R3.2, R6.2: now also U6.3 (+)
- net at C15.2, R17.2, R20.2: now also U7.3 (+)
- net at C6.1, R11.2, R12.1: now also U6.4 (-)
- net at C6.2, R12.2, R8.1: now also U6.1
- net at C21.1, R24.2, R26.1: now also U7.4 (-)
Changed lines of the file:
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@@
 		)
 		(property "Value" "NSI6801"
-			(at 143.51 81.28 0)
+			(at 141.224 98.044 0)
 			(effects
 				(font
 					(size 1.27 1.27)
 				)
-				(hide yes)
 			)
 		)
@@
 		)
 		(property "Value" "UWF1205S-3WR3"
-			(at 81.28 111.76 0)
+			(at 79.756 95.758 0)
 			(effects
 				(font
-					(size 1.8288 1.8288)
+					(size 1.27 1.27)
 				)
 				(justify left bottom)
-				(hide yes)
 			)
 		)
@@
 	)
 	(symbol
-		(lib_id "Amplifier_Operational:LMV321")
-		(at 275.59 73.66 0)
-		(unit 1)
-		(exclude_from_sim no)
-		(in_bom yes)
-		(on_board yes)
-		(dnp no)
-		(property "Reference" "U2"
-			(at 278.13 69.85 0)
-			(effects
-				(font
-					(size 1.27 1.27)
-				)
-			)
-		)
-		(property "Value" "LMV321IDBVR"
-			(at 280.67 77.47 0)
-			(effects
-				(font
-					(size 1.27 1.27)
-				)
-			)
-		)
-		(property "Footprint" "Package_TO_SOT_SMD:SOT-23-5"
-			(at 275.59 73.66 0)
-			(effects
-				(font
-					(size 1.27 1.27)
-				)
-				(justify left)
-				(hide yes)
-			)
-		)
-		(property "Datasheet" "http://www.ti.com/lit/ds/symlink/lmv324.pdf"
-			(at 275.59 73.66 0)
-			(effects
-				(font
-					(size 1.27 1.27)
-				)
-				(hide yes)
-			)
-		)
-		(property "Description" ""
-			(at 275.59 73.66 0)
-			(effects
-				(font
-					(size 1.27 1.27)
-				)
-				(hide yes)
-			)
-		)
-		(pin "2"
-		)
-		(pin "5"
-		)
-		(pin "1"
-		)
-		(pin "3"
-		)
-		(pin "4"
-		)
-		(instances
-			(project "Precharge_Nauka"
-				(path "/4c7ed5b8-d5c3-4df8-8b69-45d446422c1d"
-					(reference "U2")
-					(unit 1)
-				)
-			)
-		)
-	)
-	(symbol
 		(lib_id "Device:R")
 		(at 101.6 250.19 270)
@@
 	)
 	(symbol
+		(lib_id "Amplifier_Operational:OPA333xxDBV")
+		(at 275.59 73.66 0)
+		(unit 1)
+		(exclude_from_sim no)
+		(in_bom yes)
+		(on_board yes)
+		(dnp no)
+		(property "Reference" "U6"
+			(at 287.02 67.2045 0)
+			(effects
+				(font
+					(size 1.27 1.27)
+				)
+			)
+		)
+		(property "Value" "OPA333xxDBV"
+			(at 281.94 69.85 0)
+			(effects
+				(font
+					(size 1.27 1.27)
+				)
+			)
+		)
+		(property "Footprint" "Package_TO_SOT_SMD:SOT-23-5"
+			(at 273.05 78.74 0)
+			(effects
+				(font
+					(size 1.27 1.27)
+				)
+				(justify left)
+				(hide yes)
+			)
+		)
+		(property "Datasheet" "http://www.ti.com/lit/ds/symlink/opa333.pdf"
+			(at 275.59 68.58 0)
+			(effects
+				(font
+					(size 1.27 1.27)
+				)
+				(hide yes)
+			)
+		)
+		(property "Description" "Single 1.8V, microPower, CMOS Operational Amplifiers, Zero-Drift Series, SOT-23-5"
+			(at 275.59 73.66 0)
+			(effects
+				(font
+					(size 1.27 1.27)
+				)
+				(hide yes)
+			)
+		)
+		(pin "5"
+		)
+		(pin "2"
+		)
+		(pin "3"
+		)
+		(pin "1"
+		)
+		(pin "4"
+		)
+		(instances
+			(project ""
+				(path "/4c7ed5b8-d5c3-4df8-8b69-45d446422c1d"
+					(reference "U6")
+					(unit 1)
+				)
+			)
+		)
+	)
+	(symbol
 		(lib_id "Transistor_FET:2N7002")
 		(at 128.27 62.23 0)
@@
 	)
 	(symbol
+		(lib_id "Amplifier_Operational:OPA333xxDBV")
+		(at 275.59 118.11 0)
+		(unit 1)
+		(exclude_from_sim no)
+		(in_bom yes)
+		(on_board yes)
+		(dnp no)
+		(property "Reference" "U7"
+			(at 287.02 111.6545 0)
+			(effects
+				(font
+					(size 1.27 1.27)
+				)
+			)
+		)
+		(property "Value" "OPA333xxDBV"
+			(at 282.956 114.3 0)
+			(effects
+				(font
+					(size 1.27 1.27)
+				)
+			)
+		)
+		(property "Footprint" "Package_TO_SOT_SMD:SOT-23-5"
+			(at 273.05 123.19 0)
+			(effects
+				(font
+					(size 1.27 1.27)
+				)
+				(justify left)
+				(hide yes)
+			)
+		)
+		(property "Datasheet" "http://www.ti.com/lit/ds/symlink/opa333.pdf"
+			(at 275.59 113.03 0)
+			(effects
+				(font
+					(size 1.27 1.27)
+				)
+				(hide yes)
+			)
+		)
+		(property "Description" "Single 1.8V, microPower, CMOS Operational Amplifiers, Zero-Drift Series, SOT-23-5"
+			(at 275.59 118.11 0)
+			(effects
+				(font
+					(size 1.27 1.27)
+				)
+				(hide yes)
+			)
+		)
+		(pin "5"
+		)
+		(pin "2"
+		)
+		(pin "3"
+		)
+		(pin "1"
+		)
+		(pin "4"
+		)
+		(instances
+			(project "Precharge_Nauka"
+				(path "/4c7ed5b8-d5c3-4df8-8b69-45d446422c1d"
+					(reference "U7")
+					(unit 1)
+				)
+			)
+		)
+	)
+	(symbol
 		(lib_id "Device:R")
 		(at 127 267.97 270)
@@
 	)
 	(symbol
-		(lib_id "Amplifier_Operational:LMV321")
-		(at 275.59 118.11 0)
-		(unit 1)
-		(exclude_from_sim no)
-		(in_bom yes)
-		(on_board yes)
-		(dnp no)
-		(property "Reference" "U4"
-			(at 278.13 114.3 0)
-			(effects
-				(font
-					(size 1.27 1.27)
-				)
-			)
-		)
-		(property "Value" "LMV321IDBVR"
-			(at 280.67 121.92 0)
-			(effects
-				(font
-					(size 1.27 1.27)
-				)
-			)
-		)
-		(property "Footprint" "Package_TO_SOT_SMD:SOT-23-5"
-			(at 275.59 118.11 0)
-			(effects
-				(font
-					(size 1.27 1.27)
-				)
-				(justify left)
-				(hide yes)
-			)
-		)
-		(property "Datasheet" "http://www.ti.com/lit/ds/symlink/lmv324.pdf"
-			(at 275.59 118.11 0)
-			(effects
-				(font
-					(size 1.27 1.27)
-				)
-				(hide yes)
-			)
-		)
-		(property "Description" ""
-			(at 275.59 118.11 0)
-			(effects
-				(font
-					(size 1.27 1.27)
-				)
-				(hide yes)
-			)
-		)
-		(pin "2"
-		)
-		(pin "5"
-		)
-		(pin "1"
-		)
-		(pin "3"
-		)
-		(pin "4"
-		)
-		(instances
-			(project "Precharge_Nauka"
-				(path "/4c7ed5b8-d5c3-4df8-8b69-45d446422c1d"
-					(reference "U4")
-					(unit 1)
-				)
-			)
-		)
-	)
-	(symbol
 		(lib_id "Device:R")
 		(at 152.4 273.05 270)
@@
 		)
 		(property "Value" "UWF1215S-3WR3"
-			(at 81.28 132.08 0)
+			(at 86.868 137.668 0)
 			(effects
 				(font
-					(size 1.8288 1.8288)
+					(size 1.27 1.27)
 				)
 				(justify left bottom)
-				(hide yes)
 			)
 		)

Commit message: VER1.0: подготовил файлы для производства v1.0
Parts:
- added H1, H2: (no value), MountingHole:MountingHole_4.3mm_M4, symbol Mechanical:MountingHole
- C1, C10, C11, C12, C13, C14, C15, C16, C17, C18, C19, C2, C20, C21, C22, C3, C4, C5, C6, C7, C9: Description P/N (none) -> Capacitor SMD 50V
- D1: value NSI6801 -> (none); Description P/N (none) -> Gate Driver; Product Name (none) -> NSI6801
- D2: value UWF1205S-3WR3 -> (none); Description P/N (none) -> DC/DC; Product Name (none) -> UWF1205S-3WR3
- D3: value UWF1215S-3WR3 -> (none); Description P/N (none) -> DC/DC; Product Name (none) -> UWF1215S-3WR3
- J1: value Conn_02x03_Top_Bottom -> (none); Description P/N (none) -> Connector; Product Name (none) -> SCT3001WV-2x03P
- J2, J3, J4: value Conn_01x01 -> (none); now left out of the parts list
- L1, L2: Description P/N (none) -> Inductor SMD; Product Name (none) -> LQH43CN220K03L
- Q1, Q6: value 2N7002 -> (none); Description P/N (none) -> MosFET npn; Product Name (none) -> 2N7002
- Q2, Q3, Q4, Q5: value C2M0280120D -> (none); Description P/N (none) -> SiC Mosfet; Product Name (none) -> C2M0280120D
- R1, R10, R100, R101, R102, R103, R104, R105, R106, R107, R108, R109, R11, R110, R111, R112, R113, R114, R115, R116, R117, R118, R119, R12, R120, R121, R122, R123, R124, R125, R126, R127, R128, R129, R13, R130, R131, R132, R133, R134, R135, R136, R137, R138, R139, R14, R140, R141, R142, R143, R144, R145, R146, R147, R148, R149, R15, R150, R151, R152, R153, R154, R155, R156, R157, R158, R159, R16, R160, R161, R162, R163, R164, R165, R166, R167, R168, R169, R17, R170, R171, R172, R173, R174, R175, R176, R177, R178, R179, R18, R180, R181, R182, R183, R184, R185, R186, R187, R188, R189, R19, R190, R191, R192, R193, R194, R195, R196, R197, R198, R199, R2, R20, R200, R201, R202, R203, R21, R22, R23, R24, R25, R26, R27, R28, R29, R3, R30, R31, R32, R33, R34, R35, R36, R37, R38, R39, R4, R40, R41, R42, R43, R44, R45, R46, R47, R48, R49, R5, R50, R51, R52, R53, R54, R55, R56, R57, R58, R59, R6, R60, R61, R62, R63, R64, R65, R66, R67, R68, R69, R7, R70, R71, R72, R73, R74, R75, R76, R77, R78, R79, R8, R80, R81, R82, R83, R84, R85, R86, R87, R88, R89, R9, R90, R91, R92, R93, R94, R95, R96, R97, R98, R99: Description P/N (none) -> Resistor SMD
- U1: value TS3702IDT -> (none); Description P/N (none) -> Comparator; Product Name (none) -> TS3702IDT
- U3: value 74LVC1G08 -> (none); Description P/N (none) -> AND; Product Name (none) -> 74LVC1G08
- U5: value PC817 -> (none); Description P/N (none) -> Optocoupler; Product Name (none) -> PC817
- U6, U7: value OPA333xxDBV -> (none); Description P/N (none) -> Op-Amp; Product Name (none) -> OPA333xxDBV
